Commit message: fix imu dumping

File: scout_gazebo/urdf/base.xacro (robot description, xacro)
@@ -10,4 +10,5 @@
     <xacro:property name="track" value="0.58306" />   <!-- track————车轮间距 -->
     <xacro:property name="wheel_vertical_offset" value="-0.0702" />
+    <!-- <xacro:property name="wheel_vertical_offset" value="0.5" /> -->
     <xacro:property name="wheel_length" value="1.1653e-01" />
     <xacro:property name="wheel_radius" value="1.6459e-01" />
@@ -26,8 +27,8 @@
     <!-- <xacro:include filename="$(find scout_gazebo)/urdf/sensor_camera.xacro" /> -->
     <!-- D435i RGB-D相机相关 -->
-    <xacro:include filename="$(find realsense_ros_gazebo)/xacro/depthcam.xacro"/>
+    <!-- <xacro:include filename="$(find realsense_ros_gazebo)/xacro/depthcam.xacro"/>
     <xacro:realsense_d435 sensor_name="camera" parent_link="base_link" rate="30.0">
     <origin rpy="0 0 0" xyz="0 0 0.3"/>
-    </xacro:realsense_d435>
+    </xacro:realsense_d435> -->
     <!-- VLP16 激光雷达 -->
     <xacro:include filename="$(find scout_gazebo)/urdf/laser_support.xacro" />
@@ -40,4 +41,5 @@
     <xacro:imu sensor_name="imu" parent_link="base_link">
     <origin rpy="0 0 0" xyz="-0.03 0 ${base_z_size/2}"/>
+    <!-- <origin rpy="0 0 0" xyz="-0.03 0 -0.5"/> -->
     </xacro:imu>
     <!-- 机器人导航控制模块 -->
@@ -67,7 +69,7 @@
     <link name="inertial_link">
         <inertial>
-            <mass value="40" />
+            <mass value="400" />
             <origin xyz="0.0 0.0 0.0" />
-            <inertia ixx="2.288641" ixy="0" ixz="0" iyy="5.103976" iyz="0" izz="3.431465" />
+            <inertia ixx="02.288641" ixy="0" ixz="0" iyy="05.103976" iyz="0" izz="03.431465" />
         </inertial>
     </link>
@@ -80,5 +82,5 @@
     <!-- wheel labeled from 0 to 3, conter-clockwise, starting from front right wheel -->
     <!-- motor 1 and 2 (left side) are mechanically installed in a reversed direction -->
-    <xacro:scout_wheel_type1 wheel_prefix="front_right">
+    <!-- <xacro:scout_wheel_type1 wheel_prefix="front_right">
         <origin xyz="${wheelbase/2} ${-track/2} ${wheel_vertical_offset}" rpy="3.14 0 0" />
     </xacro:scout_wheel_type1>
@@ -91,4 +93,26 @@
     <xacro:scout_wheel_type2 wheel_prefix="rear_right">
         <origin xyz="${-wheelbase/2} ${-track/2} ${wheel_vertical_offset}" rpy="3.14 0 0" />
+    </xacro:scout_wheel_type2> -->
+    <!-- <xacro:scout_wheel_type1 wheel_prefix="front_right">
+        <origin xyz="${wheelbase} ${-track} ${wheel_vertical_offset}" rpy="3.14 0 0" />
+    </xacro:scout_wheel_type1>
+    <xacro:scout_wheel_type2 wheel_prefix="front_left">
+        <origin xyz="${wheelbase} ${track} ${wheel_vertical_offset}" rpy="0 0 0" />
     </xacro:scout_wheel_type2>
+    <xacro:scout_wheel_type1 wheel_prefix="rear_left">
+        <origin xyz="${-wheelbase} ${track} ${wheel_vertical_offset}" rpy="0 0 0" />
+    </xacro:scout_wheel_type1>
+    <xacro:scout_wheel_type2 wheel_prefix="rear_right">
+        <origin xyz="${-wheelbase} ${-track} ${wheel_vertical_offset}" rpy="3.14 0 0" />
+    </xacro:scout_wheel_type2> -->
+    <!-- <xacro:macro name="laser_sensor">
+        <link name="scan">
+            <pose>0.2 0 0.1 0 0 0</pose>
+        </link>
+        <joint name="base_link_to_scan" type="fixed">
+            <parent link="base_link"/>
+            <child link="scan"/>
+            <origin xyz="0.2 0 0.1" rpy="0 0 0"/>
+        </joint>
+    </xacro:macro> -->
 </robot>

File: scout_gazebo/urdf/imu.xacro (robot description, xacro)
@@ -6,5 +6,5 @@
         <xacro:property name="imu_offset_z" value="0.2" />
         <xacro:property name="imu_size"     value="0.05" />
-        <xacro:property name="imu_m" value="0.01" /> <!-- imu质量 -->
+        <xacro:property name="imu_m" value="0.000000001" /> <!-- imu质量 0.01 -->
         <!-- imu -->
         <joint name="imutobase" type="fixed">
@@ -45,5 +45,5 @@
                 <bodyName>imu_base</bodyName>
                 <updateRateHZ>100.0</updateRateHZ>
-                <gaussianNoise>0.01</gaussianNoise>
+                <gaussianNoise>0.001</gaussianNoise>
                 <xyzOffset>0 0 0</xyzOffset>
                 <rpyOffset>0 0 0</rpyOffset>

File: scout_gazebo/urdf/laser_support.xacro (robot description, xacro)
@@ -7,5 +7,5 @@
     <xacro:property name="support_y_size" value="0.0" /> <!-- 支架安装的y坐标 -->
     <xacro:property name="support_z_size" value="${base_z_size}" /> <!-- 支架安装的z坐标:底盘高度 / 2 + 支架高度 / 2  -->
-    <xacro:property name="support_m" value="0.02" /> <!-- 支架质量 -->
+    <xacro:property name="support_m" value="0.000000001" /> <!-- 支架质量 0.02 -->
     <link name="support">
         <visual>

File: scout_gazebo/urdf/move.xacro (robot description, xacro)
@@ -1,40 +1,4 @@
 <?xml version="1.0"?>
 <robot name="my_car_move" xmlns:xacro="http://wiki.ros.org/xacro">
-    <!-- 传动实现:用于连接控制器与关节 -->
-    <xacro:macro name="joint_trans" params="joint_name">
-        <!-- Transmission is important to link the joints and the controller -->
-        <transmission name="${joint_name}_trans">
-            <type>transmission_interface/SimpleTransmission</type>
-            <joint name="${joint_name}">
-                <hardwareInterface>hardware_interface/VelocityJointInterface</hardwareInterface>
-            </joint>
-            <actuator name="${joint_name}_motor">
-                <hardwareInterface>hardware_interface/VelocityJointInterface</hardwareInterface>
-                <mechanicalReduction>1</mechanicalReduction>
-            </actuator>
-        </transmission>
-    </xacro:macro>
-    <!-- 每一个驱动轮都需要配置传动装置 -->
-    <xacro:joint_trans joint_name="front_left_wheel" />
-    <xacro:joint_trans joint_name="front_right_wheel" />
-    <xacro:joint_trans joint_name="rear_left_wheel" />
-    <xacro:joint_trans joint_name="rear_right_wheel" />
-    <!-- 控制器 -->
-    <gazebo>
-  		<plugin name="skid_steer_drive_controller" filename="libgazebo_ros_skid_steer_drive.so">
-    		<updateRate>100.0</updateRate>
-    		<robotNamespace>/</robotNamespace>
-    		<leftFrontJoint>front_left_wheel</leftFrontJoint>
-    		<rightFrontJoint>front_right_wheel</rightFrontJoint>
-    		<leftRearJoint>rear_left_wheel</leftRearJoint>
-    		<rightRearJoint>rear_right_wheel</rightRearJoint>
-    		<wheelSeparation>${track}</wheelSeparation>
-    		<wheelDiameter>${wheel_radius * 2}</wheelDiameter>
-    		<robotBaseFrame>base_link</robotBaseFrame>
-    		<torque>20</torque>
-    		<topicName>cmd_vel</topicName>
-    		<broadcastTF>false</broadcastTF>
-  		</plugin>
-	</gazebo>
   <gazebo>
     <plugin name="object_controller" filename="libgazebo_ros_planar_move.so">
@@ -44,4 +8,5 @@
       <odometryRate>20.0</odometryRate>
       <robotBaseFrame>base_link</robotBaseFrame>
+      <ground_truth>true</ground_truth>
     </plugin>
   </gazebo>

File: scout_gazebo/urdf/scout_wheel_type1.xacro (robot description, xacro)
@@ -41,4 +41,5 @@
                 <geometry>
                     <cylinder length="${wheel_length}" radius="${wheel_radius}" />
+                    <!-- <box size="0.02 ${2 * wheel_radius} ${wheel_length}"/>  -->
                 </geometry>
             </collision>
@@ -49,4 +50,5 @@
             <xacro:insert_block name="joint_pose"/>
             <axis xyz="0 -1 0" rpy="0 0 0" />
+            <!-- <dynamics damping="0.1" friction="0.2"/> -->
         </joint>
     </xacro:macro>

File: scout_gazebo/urdf/scout_wheel_type2.xacro (robot description, xacro)
@@ -41,4 +41,5 @@
                 <geometry>
                     <cylinder length="${wheel_length}" radius="${wheel_radius}" />
+                    <!-- <box size="0.02 ${2 * wheel_radius} ${wheel_length}"/>  -->
                 </geometry>
             </collision>
@@ -49,4 +50,5 @@
             <xacro:insert_block name="joint_pose"/>
             <axis xyz="0 -1 0" rpy="0 0 0" />
+            <!-- <dynamics damping="0.1" friction="0.2"/> -->
         </joint>
     </xacro:macro>

File: velodyne_simulator/velodyne_description/urdf/VLP-16.urdf.xacro (robot description, xacro)
@@ -10,9 +10,10 @@
     <link name="${name}_base_link">
       <inertial>
-        <mass value="0.83"/>
+        <mass value="0.00000001"/> <!-- 0.83-->
         <origin xyz="0 0 0.03585"/>
-        <inertia ixx="${(0.83 * (3.0*0.0516*0.0516 + 0.0717*0.0717)) / 12.0}" ixy="0" ixz="0"
+        <!-- <inertia ixx="${(0.83 * (3.0*0.0516*0.0516 + 0.0717*0.0717)) / 12.0}" ixy="0" ixz="0"
           iyy="${(0.83 * (3.0*0.0516*0.0516 + 0.0717*0.0717)) / 12.0}" iyz="0"
-          izz="${0.5 * 0.83 * (0.0516*0.0516)}"/>
+          izz="${0.5 * 0.83 * (0.0516*0.0516)}"/> -->
+        <inertia ixx="0" ixy="0" ixz="0" iyy="0" iyz="0" izz="0"/>
       </inertial>
       <visual>
@@ -40,5 +41,5 @@
     <link name="${name}">
       <inertial>
-        <mass value="0.01"/>
+        <mass value="0"/> <!-- 0.01 -->
         <origin xyz="0 0 0"/>
         <inertia ixx="1e-7" ixy="0" ixz="0" iyy="1e-7" iyz="0" izz="1e-7"/>
